Commit message: multiple optimsations run

File: slipstick_rig.urdf (robot description, URDF)
Before this commit: robot slip_stick_rig, 6 links, 5 joints
Links:
- link foot: geometry collision box size=0.02 0.05 0.005; collision box size=0.02 0.05 0.005
- link leg: mass 0.15 -> 0.25; geometry visual box size=0.02 0.02 0.5; visual cylinder length=0.02 radius=0.01
- link mass: mass 2.0 -> 5.0; geometry visual sphere radius=0.055
Joints:
- removed joint world_to_x_prismatic
- removed joint x_to_z_prismatic
- added joint x_prismatic: type prismatic, parent world, child x_stage, origin xyz=0 0 0 rpy=0 0 0, axis 1 0 0, limit lower=0.0 upper=1.2 effort=1e6 velocity=5.0
- added joint z_prismatic: type prismatic, parent x_stage, child z_stage, origin xyz=0 0 0 rpy=0 0 0, axis 0 0 1, limit lower=-1.2 upper=-0.0 effort=1e6 velocity=5.0
- joint ankle_y: origin xyz=0 0 -0.15 rpy=0 0 0 -> xyz=0 0 -0.25 rpy=0 0 0
- joint leg_to_mass_weld: origin xyz=0 0 0.15 rpy=0 0 0 -> xyz=0 0 0.25 rpy=0 0 0
- joint z_to_leg_fixed: origin xyz=0 0 0.15 rpy=0 0 0 -> xyz=0 0 0.25 rpy=0 0 0

Commit message: new sims and added permanent hook

File: slipstick_rig.urdf (robot description, URDF)
Before this commit: robot slip_stick_rig, 6 links, 5 joints
Links:
- link foot: geometry collision box size=0.0075 0.05 0.007; collision box size=0.02 0.05 0.005
Joints:
- joint z_prismatic: limit lower=-1.2 upper=-0.0 effort=1e6 velocity=5.0 -> lower=-1.2 upper=5 effort=1e6 velocity=5.0
